File: pcbs/eyesunicolor/eyesunicolor.kicad_pcb (KiCad board)
At the start: 2 copper layers, 203.5 x 96.5 mm, 55 parts, among them J1 SUPP28, J2 SUPP28, P1 CONN_5X2, P2 CONN_5X2, P3 CONN_5X2

Commit message: agrego nuestros nombres en el PCB
Other:
- board text added: "JM-AB"
Changed lines of the file:
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@@
     (area 48.667999 54.001999 252.322001 150.634701)
     (thickness 1.6)
-    (drawings 44)
+    (drawings 48)
     (tracks 353)
     (zones 0)
@@
     (visible_elements 7FFFFFFF)
     (pcbplotparams
-      (layerselection 268468225)
+      (layerselection 32769)
       (usegerberextensions false)
       (excludeedgelayer true)
@@
       (hpglpendiameter 15)
       (hpglpenoverlay 2)
-      (psnegative false)
+      (psnegative true)
       (psa4output false)
       (plotreference true)
@@
       (padsonsilk false)
       (subtractmaskfromsilk false)
-      (outputformat 1)
+      (outputformat 2)
       (mirror false)
-      (drillshape 0)
+      (drillshape 2)
       (scaleselection 1)
       (outputdirectory ""))
@@
     )
   )
+  (gr_text JM-AB (at 202.184 86.106 270) (layer B.Cu)
+    (effects (font (size 2.032 2.032) (thickness 0.508)) (justify mirror))
+  )
+  (gr_text JM-AB (at 202.184 86.106 270) (layer F.Cu)
+    (effects (font (size 2.032 2.032) (thickness 0.508)))
+  )
+  (gr_text JM-AB (at 98.806 86.106 90) (layer F.Cu)
+    (effects (font (size 2.032 2.032) (thickness 0.508)))
+  )
+  (gr_text JM-AB (at 98.806 86.106 90) (layer B.Cu)
+    (effects (font (size 2.032 2.032) (thickness 0.508)) (justify mirror))
+  )
   (gr_circle (center 247.142 145.542) (end 249.174 145.542) (layer Edge.Cuts) (width 0.0254))

Commit message: Arreglo la falla de VCC
Parts:
- removed 1PIN (x12): P***, 1pin
Routing:
- net VCC: track 8.13 -> 74.1 mm, vias 0 -> 2
- net GND: track 4.06 -> 50.4 mm, vias 0 -> 2
- net /XLAT_D: track 134.3 -> 121.6 mm
- net /SCLK_D: track 141.0 -> 137.3 mm
- net N-0000045: track 33.8 -> 35.1 mm
- net N-0000048: track 36.5 -> 35.7 mm
