File: pcbs/control_remoto/Parlante.sch (KiCad schematic (older format))
At the start: 12 parts, among them J1 JACK_TRS_6PINS

Commit message: agrego algunos cambios en el control y casi termino la placa principal
Connections:
- net GND: now also C?.2
- net VCC2: now also C?.1, L?.2; no longer C?.2
- net In renamed IN
- net VCC1 renamed VCC
Other:
- moved on the sheet: C6, C7, C8, C9, C?, J1, L?, R11, R12, R7, RV3, U?

Commit message: completo el esquematico del control y asigno footprints
Parts:
- removed C6: C, symbol C
- removed C9: 250u, symbol C
- added C11, C12: 33n, Capacitors_ThroughHole:C_Disc_D3_P2.5, symbol C
- added C13: 1u, Capacitors_ThroughHole:C_Disc_D3_P2.5, symbol C
- added C6: 10u, Capacitors_ThroughHole:C_Radial_D5_L6_P2.5, symbol CP_Small
- added C9: 220u, Capacitors_ThroughHole:C_Radial_D5_L6_P2.5, symbol CP_Small
- added L2: 1u, Resistors_ThroughHole:Resistor_Horizontal_RM10mm, symbol INDUCTOR
- added R13, R14: 1k, Resistors_ThroughHole:Resistor_Horizontal_RM10mm, symbol R
- added U6: TL082, Sockets_DIP:DIP-8__300_ELL, symbol TL082
- C14: renamed from C?; footprint (none) -> Capacitors_ThroughHole:C_Disc_D3_P2.5
- C7, C8: footprint (none) -> Capacitors_ThroughHole:C_Disc_D3_P2.5
- J1: footprint (none) -> Pin_Headers:Pin_Header_Angled_1x06
- L3: renamed from L?; footprint (none) -> Resistors_ThroughHole:Resistor_Horizontal_RM10mm
- R11, R12, R7: footprint (none) -> Resistors_ThroughHole:Resistor_Horizontal_RM10mm
- RV3: footprint (none) -> Pin_Headers:Pin_Header_Straight_1x03
- U7: renamed from U?; footprint (none) -> Sockets_DIP:DIP-8__300_ELL
Connections:
- net GND: now also C11.2, C12.2, C13.2, U6.4 (V-), U6.4 (V-)
- net IN: now also R13.2
- net VCC: now also L2.1
- net at J1.2 (T), J1.3 (R): now also C9.2
- net at R7.1, U7.5: now also C9.1
- net at RV3.1: now also C6.2
- new net: R14.2, U6.1, U6.2 (-)
- new net: C11.1, R13.1, U6.3 (+)
- new net: C12.1, R14.1, U6.5 (+)
- new net: C6.1, U6.6 (-), U6.7
- new net VCC3: C13.1, L2.2, U6.8 (V+), U6.8 (V+)
Other:
- moved on the sheet: C14, C7, C8, J1, L3, R11, R12, R7, RV3, U7
