File: pcbs/control_remoto/controlremoto.kicad_pcb (KiCad board)
At the start: 2 copper layers, 56 parts, among them J1 JACK_TRS_6PINS, P1 CONN_BATT, P10 CONN_BTN04, P11 CONN_BTN09, P12 CONN_MIC, P13 DIPSWITCH, P2 CONN_BTN00, P3 CONN_BTN05, P4 CONN_BTN01, P5 CONN_BTN06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

Commit message: Placa Control remoto
Parts:
- moved C10 179.5 mm to (229.9, 69.8)
- moved P12 174.1 mm to (212.1, 78.7)
- moved R12 164.6 mm to (226.1, 82.5)
- moved RV1 163.1 mm to (194.3, 64.8), turned to 0 degrees
- moved C5 162.9 mm to (229.9, 63.5)
- moved RV2 161.5 mm to (208.3, 64.8)
- moved R5 160.0 mm to (188.0, 66.0), turned to 90 degrees
- moved U4 159.8 mm to (219.7, 67.3), turned to 270 degrees
- moved R4 152.5 mm to (226.1, 77.5)
- moved R9 152.0 mm to (201.9, 66.0), turned to 270 degrees
- moved R6 142.8 mm to (180.3, 66.0)
- moved P11 140.1 mm to (98.8, 165.4), turned to 180 degrees
- moved C3 137.1 mm to (186.7, 77.5)
- moved R10 135.8 mm to (200.7, 77.5)
- moved L1 132.3 mm to (177.8, 77.5), turned to 0 degrees
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Routing:
- net /DIPSW_7: track 0.00 -> 36.7 mm
- net +5V: track 0.00 -> 34.9 mm, vias 0 -> 2
- net /DIPSW_8: track 0.00 -> 34.4 mm
- net /DIPSW_5: track 0.00 -> 30.6 mm
- net /DIPSW_4: track 0.00 -> 30.6 mm
- net /DIPSW_6: track 0.00 -> 29.8 mm
- net Net-(C1-Pad1): track 0.00 -> 27.1 mm
- net /DIPSW_3: track 0.00 -> 11.4 mm
- net /DIPSW_2: track 0.00 -> 11.4 mm
- net /DIPSW_1: track 0.00 -> 11.4 mm
- net +BATT: track 0.00 -> 10.2 mm
- net Net-(R2-Pad1): track 0.00 -> 8.42 mm
- added copper zone on B.Cu, net GND
Other:
- board outline added: 200.7 x 61 mm
- net class Default: clearance 0.2 -> 0.3048; trace_width 0.25 -> 0.3048; via_dia 0.6 -> 1.524; via_drill 0.4 -> 0.7
- rule trace_clearance: 0.2 -> 0.3048

Commit message: Placa control
Parts:
- moved R1 10.2 mm to (113.0, 64.8), turned to 0 degrees
- moved R3 1.02 mm to (113.0, 71.1), turned to 0 degrees
Routing:
- net +3V3: track 0.00 -> 106.3 mm
- net +5V: track 34.9 -> 108.5 mm
- net /ZIGBIT_RX: track 0.00 -> 69.1 mm
- net /ZIGBIT_TX: track 0.00 -> 65.5 mm
- net /SCL: track 0.00 -> 43.6 mm
- net /ZB_RESET: track 0.00 -> 42.5 mm
- net /SDA: track 0.00 -> 38.1 mm
- net /Parlante/IN: track 0.00 -> 16.8 mm

Commit message: Placa control
Parts:
- moved R6 47.1 mm to (225.6, 79.2), turned to 270 degrees
- moved C5 46.3 mm to (184.9, 74.4)
- moved C3 33.8 mm to (220.5, 79.2), turned to 270 degrees
- moved C4 31.1 mm to (188.2, 83.1)
- moved R8 28.8 mm to (202.7, 67.8), turned to 270 degrees
- moved C8 27.2 mm to (194.3, 105.9)
- moved C6 26.9 mm to (192.8, 114.3), turned to 0 degrees
- moved R5 26.6 mm to (194.8, 91.7), turned to 180 degrees
- moved RV1 24.7 mm to (184.9, 87.6), turned to 90 degrees
- moved RV3 24.4 mm to (200.2, 114.3), turned to 90 degrees
- moved L1 24.0 mm to (193.3, 95.8)
- moved U4 21.5 mm to (202.2, 79.8), turned to 180 degrees
- moved R7 21.0 mm to (202.9, 105.9), turned to 180 degrees
- moved C10 20.7 mm to (213.4, 82.3)
- moved U6 18.4 mm to (179.8, 110.2), turned to 180 degrees
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Routing:
- net +5V: track 108.5 -> 227.7 mm
- net /MIC: track 0.00 -> 58.0 mm
- net Net-(C3-Pad1): track 0.00 -> 35.2 mm
- net Net-(R5-Pad2): track 0.00 -> 34.4 mm
- net Net-(R6-Pad1): track 0.00 -> 30.0 mm
- net /Parlante/VCC3: track 0.00 -> 25.8 mm
- net /VCC2: track 0.00 -> 25.3 mm
- net Net-(RV3-Pad2): track 0.00 -> 25.2 mm
- net Net-(C7-Pad2): track 0.00 -> 24.1 mm
- net Net-(C9-Pad1): track 0.00 -> 22.8 mm
- net /Parlante/VCC2: track 0.00 -> 17.4 mm
- net Net-(C6-Pad1): track 0.00 -> 17.3 mm
- net Net-(C11-Pad1): track 0.00 -> 17.2 mm
- net Net-(R9-Pad2): track 0.00 -> 16.9 mm
- net Net-(C12-Pad1): track 0.00 -> 15.5 mm
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
Commit message: primera version del control, falta verificar footprint
Parts:
- C9: value 250u -> 220u
- moved P8 114.7 mm to (66.0, 65.4), turned to 0 degrees
- moved P3 113.1 mm to (167.0, 64.1), turned to 270 degrees
- moved P7 111.5 mm to (167.0, 73.0), turned to 270 degrees
- moved P11 107.8 mm to (167.0, 81.9), turned to 270 degrees
- moved P5 106.4 mm to (167.0, 68.6), turned to 270 degrees
- moved P4 105.1 mm to (66.0, 87.0), turned to 0 degrees
- moved P6 104.8 mm to (66.0, 76.2), turned to 0 degrees
- moved P9 104.5 mm to (167.0, 77.5), turned to 270 degrees
- moved P2 97.0 mm to (66.0, 97.8), turned to 0 degrees
- moved P10 75.5 mm to (66.0, 108.6), turned to 0 degrees
- moved U2 5.75 mm to (54.0, 80.6)
- moved R2 5.75 mm to (54.0, 62.9)
- moved C1 5.75 mm to (51.4, 101.0)
- moved C2 5.75 mm to (59.1, 101.0)
- moved P1 5.75 mm to (50.2, 113.7)
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Connections:
- J1 pad 2: Net-(C9-Pad1) -> Net-(C9-Pad2)
- J1 pad 3: Net-(C9-Pad1) -> Net-(C9-Pad2)
- R7 pad 1: Net-(C9-Pad2) -> Net-(C9-Pad1)
- U3 pad 10: /ACEL_INT2 -> (no net)
- U3 pad 11: /BTN_08 -> /BTN_04
- U3 pad 12: /BTN_09 -> (no net)
- U3 pad 22: (no net) -> /BTN_09
- U3 pad 23: /BTN_07 -> /BTN_08
- U3 pad 24: /BTN_06 -> /BTN_07
- U3 pad 25: /BTN_05 -> /BTN_06
- U3 pad 26: /BTN_04 -> /BTN_05
- U3 pad 29: (no net) -> /ACEL_INT2
- U3 pad 30: (no net) -> /ACEL_INT1
- U3 pad 9: /ACEL_INT1 -> (no net)
- U7 pad 5: Net-(C9-Pad2) -> Net-(C9-Pad1)
Routing:
- net /BTN_03: track 0.00 -> 146.8 mm, vias 0 -> 2
- net /BTN_02: track 0.00 -> 133.3 mm, vias 0 -> 2
- net /BTN_01: track 0.00 -> 119.5 mm, vias 0 -> 2
- net /BTN_00: track 0.00 -> 106.1 mm, vias 0 -> 2
- net /BTN_04: track 0.00 -> 85.0 mm, vias 0 -> 2
- net /ACEL_INT1: track 0.00 -> 46.7 mm, vias 0 -> 2
- net /ACEL_INT2: track 0.00 -> 38.5 mm, vias 0 -> 2
- net /BTN_05: track 0.00 -> 33.9 mm
- net /BTN_06: track 0.00 -> 29.1 mm
- net /BTN_07: track 0.00 -> 23.6 mm
- net /BTN_08: track 0.00 -> 18.5 mm
- net /BTN_09: track 0.00 -> 13.4 mm
- net Net-(C9-Pad1): track 22.8 -> 12.8 mm
- net Net-(C9-Pad2): track 15.5 -> 25.0 mm
- net +3V3: track 106.3 -> 114.0 mm
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
Commit message: actualizo las 3 placas, revisar y mandar a fabricar
Parts:
- removed R14: 1k, Resistors_ThroughHole:Resistor_Horizontal_RM10mm
- added J2: Jack-stereo-gnd, Popurri_CDR:audio-jack-stereo, F.Cu at (213.6, 112.6)
- added REF**: 1pin, Connect:1pin, F.Cu at (146.7, 65.8)
- added REF**: 1pin, Connect:1pin, F.Cu at (92.1, 108.7)
- added REF**: 1pin, Connect:1pin, F.Cu at (86.9, 66.8)
- added REF**: 1pin, Connect:1pin, F.Cu at (176.0, 63.0)
- added REF**: 1pin, Connect:1pin, F.Cu at (115.4, 82.0)
- C10, C13, C14: footprint Capacitors_ThroughHole:C_Disc_D3_P2.5 -> Capacitors_ThroughHole:C_Rect_L18_W5_P15
- C11, C12, C4, C5: footprint Capacitors_ThroughHole:C_Disc_D3_P2.5 -> Capacitors_ThroughHole:C_Rect_L7_W2_P5
- J1: value JACK_TRS_6PINS -> Jack-stereo-gnd; footprint Pin_Headers:Pin_Header_Angled_1x06 -> Popurri_CDR:audio-jack-stereo
- P12: value CONN_MIC -> CONN_01X03; footprint Connect:PINHEAD1-2 -> Socket_Strips:Socket_Strip_Straight_1x03
- R5: value 100k -> 1k
- moved L3 43.4 mm to (175.4, 75.9), turned to 90 degrees
- moved U7 40.2 mm to (183.3, 88.1), turned to 270 degrees
- moved RV1 35.4 mm to (214.4, 67.9), turned to 180 degrees
- moved RV3 32.4 mm to (174.6, 94.4), turned to 180 degrees
- moved C14 28.7 mm to (184.5, 77.0)
- moved P12 27.2 mm to (213.1, 101.9), turned to 0 degrees
- moved C5 26.7 mm to (209.2, 63.2), turned to 180 degrees
- moved C4 26.7 mm to (209.3, 66.7), turned to 180 degrees
- moved R5 23.9 mm to (172.3, 99.9), turned to 0 degrees
- moved RV2 23.8 mm to (207.0, 87.5), turned to 270 degrees
- moved R8 23.2 mm to (214.2, 87.9)
- moved J1 22.6 mm to (199.8, 112.6), turned to 90 degrees
- moved C13 21.5 mm to (187.6, 115.6)
- moved C10 20.6 mm to (193.2, 78.2), turned to 90 degrees
- moved R6 19.1 mm to (210.9, 91.6)
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Connections:
- J1 pad 3: Net-(C9-Pad2) -> Net-(J1-Pad3)
- J1 pad 4: GND -> Net-(J1-Pad4)
- J1 pad 5: Net-(J1-Pad5) -> Net-(C9-Pad2)
- P12 pad 1: GND -> /MicB
- R11 pad 2: Net-(J1-Pad5) -> Net-(J1-Pad4)
- R12 pad 2: Net-(J1-Pad6) -> Net-(J1-Pad3)
- R5 pad 1: /VCC2 -> Net-(C12-Pad1)
- RV1 pad 1: Net-(R5-Pad2) -> /VCC2
- RV1 pad 2: Net-(R5-Pad2) -> Net-(RV1-Pad2)
- U4 pad 3: Net-(R5-Pad2) -> Net-(RV1-Pad2)
- U6 pad 1: Net-(R14-Pad2) -> Net-(R5-Pad2)
- U6 pad 2: Net-(R14-Pad2) -> Net-(R5-Pad2)
Routing:
- net /VCC2: track 25.3 -> 54.4 mm, vias 0 -> 2
- net /MIC: track 58.0 -> 87.0 mm, vias 0 -> 2
- net Net-(R5-Pad2): track 34.4 -> 6.35 mm
- net Net-(C7-Pad2): track 24.1 -> 3.47 mm
- net Net-(RV3-Pad2): track 25.2 -> 5.83 mm
- net Net-(C3-Pad1): track 35.2 -> 17.4 mm
- net /Parlante/VCC3: track 26.7 -> 11.8 mm
- net Net-(J1-Pad5): track 14.4 -> 0.00 mm
- net Net-(RV1-Pad2): track 0.00 -> 14.0 mm
- net /Parlante/VCC2: track 17.4 -> 26.8 mm
- net /Parlante/IN: track 13.8 -> 4.44 mm
- net /MicB: track 0.00 -> 8.62 mm
- net Net-(J1-Pad6): track 8.21 -> 0.00 mm
- net Net-(R14-Pad2): track 7.17 -> 0.00 mm
- net Net-(J1-Pad4): track 0.00 -> 6.14 mm
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Other:
- board size 200.7 x 61 mm -> 175.5 x 61 mm
- net class Default: via_dia 1.524 -> 1.778
- rule trace_min: 0.2 -> 0.254
- rule via_min_size: 0.4 -> 0.7
- board text added: "Marciano - Control"

Commit message: cambios hechos en las placas
Connections:
- REF** pad 1: (no net) -> GND
Routing:
- added copper zone on F.Cu, net GND
Changed lines of the file:
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@@
 (kicad_pcb (version 4) (host pcbnew 0.201504141001+5596~22~ubuntu14.04.1-product)
   (general
-    (links 132)
+    (links 133)
     (no_connects 0)
-    (area 38.024999 58.344999 238.835001 119.455001)
+    (area 43.394086 57.8252 221.055001 121.1148)
     (thickness 1.6)
     (drawings 7)
@@
   )
   (setup
-    (last_trace_width 0.508)
+    (last_trace_width 0.3048)
     (user_trace_width 0.508)
     (user_trace_width 0.762)
@@
     (mod_text_size 0.000001 0.000001)
     (mod_text_width 0.15)
-    (pad_size 2.032 2.032)
-    (pad_drill 1)
+    (pad_size 2.54 2.54)
+    (pad_drill 1.5)
     (pad_to_mask_clearance 0.2)
     (aux_axis_origin 0 0)
     (visible_elements 7FFFFF7F)
     (pcbplotparams
-      (layerselection 0x00030_80000001)
+      (layerselection 0x010c0_80000001)
       (usegerberextensions false)
       (excludeedgelayer true)
@@
       (outputformat 1)
       (mirror false)
-      (drillshape 1)
+      (drillshape 0)
       (scaleselection 1)
-      (outputdirectory ""))
+      (outputdirectory output/))
   )
   (net 0 "")
@@
     )
     (fp_circle (center 0 0) (end 0 -2.286) (layer F.SilkS) (width 0.15))
-    (pad 1 thru_hole circle (at 0 0) (size 2.54 2.54) (drill 1.5) (layers *.Cu *.Mask F.SilkS))
+    (pad 1 thru_hole circle (at 0 0) (size 2.54 2.54) (drill 1.5) (layers *.Cu *.Mask F.SilkS)
+      (net 2 GND))
   )
   (module Connect:1pin (layer F.Cu)
@@
     (connect_pads (clearance 0.3048))
     (min_thickness 0.3048)
+    (fill yes (arc_segments 16) (thermal_gap 0.3048) (thermal_bridge_width 0.508))
+    (polygon
+      (pts
+        (xy 220.853 119.253) (xy 45.593 119.253) (xy 45.593 58.547) (xy 220.853 58.547)
+      )
+    )
+  )
+  (zone (net 2) (net_name GND) (layer F.Cu) (hatch edge 0.508)
+    (connect_pads (clearance 0.3048))
+    (min_thickness 0.3048)
