File: pcbs/basicmother/power.sch (KiCad schematic (older format))
At the start: 12 parts

Commit message: Actualizo esquematico de la placa principal y empiezo con el layout
Parts:
- removed C?: 2.2u, symbol C
- removed R?: 21k, symbol R
- removed U?: PTN78000W, symbol PTN78000W
- added C10: 100u, Capacitors_ThroughHole:C_Radial_D5_L6_P2.5, symbol CAPAPOL
- added C9: 22n, Capacitors_ThroughHole:C_Disc_D3_P2.5, symbol C
- added R2: 1.07k, Resistors_ThroughHole:Resistor_Horizontal_RM10mm, symbol R
- added R3: 5.62k, Resistors_ThroughHole:Resistor_Horizontal_RM10mm, symbol R
- added R4: 100k, Resistors_ThroughHole:Resistor_Horizontal_RM10mm, symbol R
- added U4: LMZ12002, Popurri_CDR:PFM7, symbol LMZ12002
- C11: renamed from C?; value 100uA -> 10u; footprint (none) -> Capacitors_ThroughHole:C_Radial_D5_L6_P2.5
- C5, C6: renamed from C?; value 100uA -> 100u; footprint (none) -> Capacitors_ThroughHole:C_Radial_D5_L6_P2.5
- C7: renamed from C?; footprint (none) -> Capacitors_ThroughHole:C_Disc_D3_P2.5
- C8: renamed from C?; value 100n -> 22n; footprint (none) -> Capacitors_ThroughHole:C_Disc_D3_P2.5
- P6, P7: renamed from P?; footprint (none) -> Pin_Headers:Pin_Header_Straight_1x02
- R1: renamed from R?; footprint (none) -> Resistors_ThroughHole:Resistor_Horizontal_RM10mm
- U3: renamed from U?; footprint (none) -> Power_CDR:PTN04050C-EUU
Connections:
- wire segments 50 -> 63
Other:
- note removed: "ceramico \nvalor minimo\nX5R o X7R"
- moved on the sheet: C11, C8

Commit message: saque el micro para el control de los ojitos y lo pase a una placa aparte, ademas agregue un doble microfono
Parts:
- P5: renamed from P6; value CONN_01X02 -> SWITCH; footprint Pin_Headers:Pin_Header_Straight_1x02 -> Socket_Strips:Socket_Strip_Straight_1x02
- P6: renamed from P7; value CONN_01X02 -> BATT; footprint Pin_Headers:Pin_Header_Straight_1x02 -> Connect:bornier2
- renumbered C5 to C1, C6 to C2, C7 to C3, C8 to C4, C9 to C5, C10 to C6, C11 to C7, R1 to R2, R2 to R3, R3 to R4, R4 to R5, U3 to U4, U4 to U5
Changed lines of the file:
@@
 	4500 3000 4500 3150
 $Comp
-L +5V #PWR033
+L +5V #PWR022
 U 1 1 54D591BB
 P 2900 3300
-F 0 "#PWR033" H 2900 3390 20  0001 C CNN
+F 0 "#PWR022" H 2900 3390 20  0001 C CNN
 F 1 "+5V" H 2900 3390 30  0000 C CNN
 F 2 "" H 2900 3300 60  0000 C CNN
@@
 	2900 3350 3050 3350
 $Comp
-L GND #PWR034
+L GND #PWR023
 U 1 1 54D591BC
 P 2550 3150
-F 0 "#PWR034" H 2550 3150 30  0001 C CNN
+F 0 "#PWR023" H 2550 3150 30  0001 C CNN
 F 1 "GND" H 2550 3080 30  0001 C CNN
 F 2 "" H 2550 3150 60  0000 C CNN
@@
 	2550 3100 2550 3150
 $Comp
-L +12V #PWR035
+L +12V #PWR024
 U 1 1 54D591BD
 P 4500 3000
-F 0 "#PWR035" H 4500 2950 20  0001 C CNN
+F 0 "#PWR024" H 4500 2950 20  0001 C CNN
 F 1 "+12V" H 4500 3100 30  0000 C CNN
 F 2 "" H 4500 3000 60  0000 C CNN
@@
 $EndComp
 $Comp
-L CAPAPOL C6
+L CAPAPOL C2
 U 1 1 54D591BF
 P 4500 3350
-F 0 "C6" H 4550 3450 40  0000 L CNN
+F 0 "C2" H 4550 3450 40  0000 L CNN
 F 1 "100u" H 4550 3250 40  0000 L CNN
 F 2 "Capacitors_ThroughHole:C_Radial_D5_L6_P2.5" H 4600 3200 30  0001 C CNN
@@
 $EndComp
 $Comp
-L CAPAPOL C5
+L CAPAPOL C1
 U 1 1 54D591C0
 P 2900 3600
-F 0 "C5" H 2950 3700 40  0000 L CNN
+F 0 "C1" H 2950 3700 40  0000 L CNN
 F 1 "100u" H 2950 3500 40  0000 L CNN
 F 2 "Capacitors_ThroughHole:C_Radial_D5_L6_P2.5" H 3000 3450 30  0001 C CNN
@@
 	2900 3800 2900 3950
 $Comp
-L GND #PWR036
+L GND #PWR025
 U 1 1 54D591C1
 P 2900 3950
-F 0 "#PWR036" H 2900 3950 30  0001 C CNN
+F 0 "#PWR025" H 2900 3950 30  0001 C CNN
 F 1 "GND" H 2900 3880 30  0001 C CNN
 F 2 "" H 2900 3950 60  0000 C CNN
@@
 	4500 3550 4500 3650
 $Comp
-L GND #PWR037
+L GND #PWR026
 U 1 1 54D591C2
 P 4500 3650
-F 0 "#PWR037" H 4500 3650 30  0001 C CNN
+F 0 "#PWR026" H 4500 3650 30  0001 C CNN
 F 1 "GND" H 4500 3580 30  0001 C CNN
 F 2 "" H 4500 3650 60  0000 C CNN
@@
 $EndComp
 $Comp
-L CONN_01X02 P6
+L CONN_01X02 P5
 U 1 1 54D591C8
 P 4000 6150
-F 0 "P6" H 4000 6300 50  0000 C CNN
-F 1 "CONN_01X02" V 4100 6150 50  0000 C CNN
-F 2 "Pin_Headers:Pin_Header_Straight_1x02" H 4000 6150 60  0001 C CNN
+F 0 "P5" H 4000 6300 50  0000 C CNN
+F 1 "SWITCH" V 4100 6150 50  0000 C CNN
+F 2 "Socket_Strips:Socket_Strip_Straight_1x02" H 4000 6150 60  0001 C CNN
 F 3 "" H 4000 6150 60  0000 C CNN
 	1    4000 6150
@@
 $EndComp
 $Comp
-L CONN_01X02 P7
+L CONN_01X02 P6
 U 1 1 54D591C7
 P 5250 6100
-F 0 "P7" H 5250 6250 50  0000 C CNN
-F 1 "CONN_01X02" V 5350 6100 50  0000 C CNN
-F 2 "Pin_Headers:Pin_Header_Straight_1x02" H 5250 6100 60  0001 C CNN
+F 0 "P6" H 5250 6250 50  0000 C CNN
+F 1 "BATT" V 5350 6100 50  0000 C CNN
+F 2 "Connect:bornier2" H 5250 6100 60  0001 C CNN
 F 3 "" H 5250 6100 60  0000 C CNN
 	1    5250 6100
@@
 	5300 5900 5300 5750
 $Comp
-L GND #PWR038
+L GND #PWR027
 U 1 1 54D591AC
 P 5050 5750
-F 0 "#PWR038" H 5050 5750 30  0001 C CNN
+F 0 "#PWR027" H 5050 5750 30  0001 C CNN
 F 1 "GND" H 5050 5680 30  0001 C CNN
 F 2 "" H 5050 5750 60  0000 C CNN
@@
 	3500 5400 4500 5400
 $Comp
-L +15V #PWR039
+L +15V #PWR028
 U 1 1 54D5A534
 P 9500 3100
-F 0 "#PWR039" H 9500 2950 60  0001 C CNN
+F 0 "#PWR028" H 9500 2950 60  0001 C CNN
 F 1 "+15V" H 9500 3240 60  0000 C CNN
 F 2 "" H 9500 3100 60  0000 C CNN
@@
 $EndComp
 $Comp
-L +15V #PWR040
+L +15V #PWR029
 U 1 1 54D5A5D0
 P 3600 5700
-F 0 "#PWR040" H 3600 5550 60  0001 C CNN
+F 0 "#PWR029" H 3600 5550 60  0001 C CNN
 F 1 "+15V" H 3600 5840 60  0000 C CNN
 F 2 "" H 3600 5700 60  0000 C CNN
@@
 	3600 5700 3600 5750
 $Comp
-L +BATT #PWR041
+L +BATT #PWR030
 U 1 1 54D5A61A
 P 4250 5700
-F 0 "#PWR041" H 4250 5550 60  0001 C CNN
+F 0 "#PWR030" H 4250 5550 60  0001 C CNN
 F 1 "+BATT" H 4250 5840 60  0000 C CNN
 F 2 "" H 4250 5700 60  0000 C CNN
@@
 	4250 5750 4250 5700
 $Comp
-L +BATT #PWR042
+L +BATT #PWR031
 U 1 1 54D5A73D
 P 5500 5700
-F 0 "#PWR042" H 5500 5550 60  0001 C CNN
+F 0 "#PWR031" H 5500 5550 60  0001 C CNN
 F 1 "+BATT" H 5500 5840 60  0000 C CNN
 F 2 "" H 5500 5700 60  0000 C CNN
@@
 	5500 5750 5500 5700
 $Comp
-L +5V #PWR043
+L +5V #PWR032
 U 1 1 54D5A841
 P 9150 2900
-F 0 "#PWR043" H 9150 2750 60  0001 C CNN
+F 0 "#PWR032" H 9150 2750 60  0001 C CNN
 F 1 "+5V" H 9150 3040 60  0000 C CNN
 F 2 "" H 9150 2900 60  0000 C CNN
@@
 $EndComp
 $Comp
-L CAPAPOL C11
+L CAPAPOL C7
 U 1 1 54D5AA9E
 P 9500 3550
-F 0 "C11" H 9550 3650 40  0000 L CNN
+F 0 "C7" H 9550 3650 40  0000 L CNN
 F 1 "10u" H 9550 3450 40  0000 L CNN
 F 2 "Capacitors_ThroughHole:C_Radial_D5_L6_P2.5" H 9600 3400 30  0001 C CNN
@@
 $EndComp
 $Comp
-L C C8
+L C C4
 U 1 1 54D5AE89
 P 7250 3800
-F 0 "C8" H 7300 3900 50  0000 L CNN
+F 0 "C4" H 7300 3900 50  0000 L CNN
 F 1 "22n" H 7300 3700 50  0000 L CNN
 F 2 "Capacitors_ThroughHole:C_Disc_D3_P2.5" H 7288 3650 30  0001 C CNN
@@
 $EndComp
 $Comp
-L C C7
+L C C3
 U 1 1 54D5AF73
 P 4900 3350
-F 0 "C7" H 4950 3450 50  0000 L CNN
+F 0 "C3" H 4950 3450 50  0000 L CNN
 F 1 "100n" H 4950 3250 50  0000 L CNN
 F 2 "Capacitors_ThroughHole:C_Disc_D3_P2.5" H 4938 3200 30  0001 C CNN
@@
 	4900 3600 4500 3600
 $Comp
-L R R1
+L R R2
 U 1 1 54D5B373
 P 4350 3900
-F 0 "R1" V 4430 3900 50  0000 C CNN
+F 0 "R2" V 4430 3900 50  0000 C CNN
 F 1 "1.35k" V 4357 3901 50  0000 C CNN
 F 2 "Resistors_ThroughHole:Resistor_Horizontal_RM10mm" V 4280 3900 30  0001 C CNN
@@
 $EndComp
 $Comp
-L PTN4050 U3
+L PTN4050 U4
 U 1 1 54D591BE
 P 3650 3350
-F 0 "U3" H 3650 3500 60  0000 C CNN
+F 0 "U4" H 3650 3500 60  0000 C CNN
 F 1 "PTN4050" H 3650 3200 60  0000 C CNN
 F 2 "Power_CDR:PTN04050C-EUU" H 3650 3350 60  0001 C CNN
@@
 	4350 4050 4350 4250
 $Comp
-L GND #PWR044
+L GND #PWR033
 U 1 1 54D5B521
 P 4350 4250
-F 0 "#PWR044" H 4350 4250 30  0001 C CNN
+F 0 "#PWR033" H 4350 4250 30  0001 C CNN
 F 1 "GND" H 4350 4180 30  0001 C CNN
 F 2 "" H 4350 4250 60  0000 C CNN
@@
 	1100 1800 1100 1600
 $Comp
-L +12V #PWR045
+L +12V #PWR034
 U 1 1 54D5BD2B
 P 1250 1600
-F 0 "#PWR045" H 1250 1550 20  0001 C CNN
+F 0 "#PWR034" H 1250 1550 20  0001 C CNN
 F 1 "+12V" H 1250 1750 30  0000 C CNN
 F 2 "" H 1250 1600 60  0000 C CNN
@@
 $EndComp
 $Comp
-L +5V #PWR046
+L +5V #PWR035
 U 1 1 54D5BD42
 P 1100 1600
-F 0 "#PWR046" H 1100 1690 20  0001 C CNN
+F 0 "#PWR035" H 1100 1690 20  0001 C CNN
 F 1 "+5V" H 1100 1750 30  0000 C CNN
 F 2 "" H 1100 1600 60  0000 C CNN
@@
 $EndComp
 $Comp
-L +15V #PWR047
+L +15V #PWR036
 U 1 1 54D5BD89
 P 1450 1600
-F 0 "#PWR047" H 1450 1450 60  0001 C CNN
+F 0 "#PWR036" H 1450 1450 60  0001 C CNN
 F 1 "+15V" H 1450 1740 60  0000 C CNN
 F 2 "" H 1450 1600 60  0000 C CNN
@@
 	1450 2450 1450 2600
 $Comp
-L GND #PWR048
+L GND #PWR037
 U 1 1 54D5C2B6
 P 1450 2600
-F 0 "#PWR048" H 1450 2600 30  0001 C CNN
+F 0 "#PWR037" H 1450 2600 30  0001 C CNN
 F 1 "GND" H 1450 2530 30  0001 C CNN
 F 2 "" H 1450 2600 60  0000 C CNN
@@
 	6350 4750 6350 2500
 $Comp
-L LMZ12002 U4
+L LMZ12002 U5
 U 1 1 551F6356
 P 8450 3400
-F 0 "U4" H 8400 3550 60  0000 C CNN
+F 0 "U5" H 8400 3550 60  0000 C CNN
 F 1 "LMZ12002" H 8550 3400 60  0000 C CNN
 F 2 "Popurri_CDR:PFM7" H 8750 3750 60  0001 C CNN
@@
 Connection ~ 9500 3250
 $Comp
-L R R4
+L R R5
 U 1 1 551F6C00
 P 8400 2900
-F 0 "R4" V 8480 2900 50  0000 C CNN
+F 0 "R5" V 8480 2900 50  0000 C CNN
 F 1 "100k" V 8400 2900 50  0000 C CNN
 F 2 "Resistors_ThroughHole:Resistor_Horizontal_RM10mm" V 8330 2900 30  0001 C CNN
@@
 Connection ~ 8450 4500
 $Comp
-L CAPAPOL C10
+L CAPAPOL C6
 U 1 1 551F6E5B
 P 9150 4150
-F 0 "C10" H 9200 4250 40  0000 L CNN
+F 0 "C6" H 9200 4250 40  0000 L CNN
 F 1 "100u" H 9200 4050 40  0000 L CNN
 F 2 "Capacitors_ThroughHole:C_Radial_D5_L6_P2.5" H 9250 4000 30  0001 C CNN
@@
 Connection ~ 9150 3650
 $Comp
-L R R3
+L R R4
 U 1 1 551F761E
 P 8100 4200
-F 0 "R3" V 8180 4200 50  0000 C CNN
+F 0 "R4" V 8180 4200 50  0000 C CNN
 F 1 "5.62k" V 8100 4200 50  0000 C CNN
 F 2 "Resistors_ThroughHole:Resistor_Horizontal_RM10mm" V 8030 4200 30  0001 C CNN
@@
 $EndComp
 $Comp
-L R R2
+L R R3
 U 1 1 551F77EF
 P 7550 4150
-F 0 "R2" V 7630 4150 50  0000 C CNN
+F 0 "R3" V 7630 4150 50  0000 C CNN
 F 1 "1.07k" V 7550 4150 50  0000 C CNN
 F 2 "Resistors_ThroughHole:Resistor_Horizontal_RM10mm" V 7480 4150 30  0001 C CNN
@@
 Connection ~ 9150 2950
 $Comp
-L C C9
+L C C5
 U 1 1 551F7BE7
 P 8100 4000
-F 0 "C9" H 8150 4100 50  0000 L CNN
+F 0 "C5" H 8150 4100 50  0000 L CNN
 F 1 "22n" H 8150 3900 50  0000 L CNN
 F 2 "Capacitors_ThroughHole:C_Disc_D3_P2.5" H 8138 3850 30  0001 C CNN
@@
 NoConn ~ 7900 3350
 $Comp
-L GND #PWR049
+L GND #PWR038
 U 1 1 5521051E
 P 8450 4550
-F 0 "#PWR049" H 8450 4550 30  0001 C CNN
+F 0 "#PWR038" H 8450 4550 30  0001 C CNN
 F 1 "GND" H 8450 4480 30  0001 C CNN
 F 2 "" H 8450 4550 60  0000 C CNN

Commit message: actualizo las 3 placas, revisar y mandar a fabricar
Parts:
- added P11: BATT, Popurri_CDR:molex_2_recto, symbol CONN_01X02
- C4, C5: footprint Capacitors_ThroughHole:C_Disc_D3_P2.5 -> Capacitors_ThroughHole:C_Rect_L7_W2_P5
Connections:
- net +BATT: now also P11.1 (P1)
- net GND: now also P11.2 (P2)
Other:
- moved on the sheet: P6
Changed lines of the file:
@@
 L CONN_01X02 P6
 U 1 1 54D591C7
-P 5250 6100
-F 0 "P6" H 5250 6250 50  0000 C CNN
-F 1 "BATT" V 5350 6100 50  0000 C CNN
-F 2 "Connect:bornier2" H 5250 6100 60  0001 C CNN
-F 3 "" H 5250 6100 60  0000 C CNN
-	1    5250 6100
+P 5250 6000
+F 0 "P6" H 5250 6150 50  0000 C CNN
+F 1 "BATT" V 5350 6000 50  0000 C CNN
+F 2 "Connect:bornier2" H 5250 6000 60  0001 C CNN
+F 3 "" H 5250 6000 60  0000 C CNN
+	1    5250 6000
 	0    1    1    0
 $EndComp
@@
 	5300 5750 5500 5750
 Wire Wire Line
-	5300 5900 5300 5750
+	5300 5800 5300 5750
 $Comp
 L GND #PWR027
@@
 	5200 5750 5050 5750
 Wire Wire Line
-	5200 5900 5200 5750
+	5200 5800 5200 5750
 Text Notes 4750 6600 1    60   ~ 0
 CONECTOR DE BATERIA
@@
 $EndComp
 Wire Wire Line
-	5500 5750 5500 5700
+	5500 5700 5500 6200
 $Comp
 L +5V #PWR032
@@
 F 0 "C4" H 7300 3900 50  0000 L CNN
 F 1 "22n" H 7300 3700 50  0000 L CNN
-F 2 "Capacitors_ThroughHole:C_Disc_D3_P2.5" H 7288 3650 30  0001 C CNN
+F 2 "Capacitors_ThroughHole:C_Rect_L7_W2_P5" H 7288 3650 30  0001 C CNN
 F 3 "" H 7250 3800 60  0000 C CNN
 	1    7250 3800
@@
 F 0 "C5" H 8150 4100 50  0000 L CNN
 F 1 "22n" H 8150 3900 50  0000 L CNN
-F 2 "Capacitors_ThroughHole:C_Disc_D3_P2.5" H 8138 3850 30  0001 C CNN
+F 2 "Capacitors_ThroughHole:C_Rect_L7_W2_P5" H 8138 3850 30  0001 C CNN
 F 3 "" H 8100 4000 60  0000 C CNN
 	1    8100 4000
@@
 	1    0    0    -1
 $EndComp
+$Comp
+L CONN_01X02 P11
+U 1 1 55360EE8
+P 5250 6400
+F 0 "P11" H 5250 6550 50  0000 C CNN
+F 1 "BATT" V 5350 6400 50  0000 C CNN
+F 2 "Popurri_CDR:molex_2_recto" H 5250 6400 60  0001 C CNN
+F 3 "" H 5250 6400 60  0000 C CNN
+	1    5250 6400
+	0    1    1    0
+$EndComp
+Wire Wire Line
+	5500 6200 5300 6200
+Connection ~ 5500 5750
+Wire Wire Line
+	5200 6200 5100 6200
+Wire Wire Line
+	5100 6200 5100 5750
+Connection ~ 5100 5750
 $EndSCHEMATC
